Commit message: la pinza funziona su gazebo e si apre/chiude con successo

File: install/robot_arms/share/robot_arms/urdf/robotiq_hande.urdf.xacro (robot description, xacro)
@@ -1,7 +1,12 @@
 <?xml version="1.0"?>
 <robot xmlns:xacro="http://ros.org/wiki/xacro">
-  <xacro:macro name="robotiq_hande"  params="prefix origin">
+  <xacro:macro name="robotiq_hande" params="prefix origin">
+    <xacro:property name="param_file" value="$(find robot_arms)/config/gripper/hande_parameters.yaml" />
+    <xacro:property name="gripper_props" value="${xacro.load_yaml(param_file)}"/>
+    <xacro:property name="mass_val" value="${gripper_props['robotiq_hande']['mass']}" />
+    <xacro:property name="ixx_val" value="${gripper_props['robotiq_hande']['inertia']['ixx']}" />
+    <xacro:property name="upper_limit" value="${gripper_props['robotiq_hande']['limits']['upper_stroke']}" />
+    <xacro:property name="max_effort" value="${gripper_props['robotiq_hande']['limits']['max_effort']}" />
     <joint name="${prefix}base_to_gripper" type="fixed">
-      <!-- <origin rpy="0 0 0" xyz="0 0 0.00248"/> -->
       <origin rpy="0 0 0" xyz="0 0 0"/>
       <parent link="${origin}"/>
@@ -9,4 +14,9 @@
     </joint>
     <link name="${prefix}base_link">
+      <inertial>
+        <origin xyz="0 0 0.046" rpy="0 0 0"/>
+        <mass value="${mass_val}"/>
+        <inertia ixx="${ixx_val}" ixy="0.0" ixz="0.0" iyy="${ixx_val}" iyz="0.0" izz="${ixx_val}"/>
+      </inertial>
       <visual>
         <origin xyz="0 0 0" rpy="0 0 0" />
@@ -26,4 +36,9 @@
     </link>
     <link name="${prefix}jaw1_link">
+      <inertial>
+        <origin xyz="0 0 0" rpy="0 0 0"/>
+        <mass value="0.01"/>
+        <inertia ixx="0.0001" ixy="0.0" ixz="0.0" iyy="0.0001" iyz="0.0" izz="0.0001"/>
+      </inertial>
       <visual>
         <origin rpy="0 0 0" xyz="0 0 0"/>
@@ -43,4 +58,9 @@
     </link>
     <link name="${prefix}jaw2_link">
+      <inertial>
+        <origin xyz="0 0 0" rpy="0 0 0"/>
+        <mass value="0.01"/>
+        <inertia ixx="0.0001" ixy="0.0" ixz="0.0" iyy="0.0001" iyz="0.0" izz="0.0001"/>
+      </inertial>
       <visual>
         <origin rpy="0 0 0" xyz="0 0 0"/>
@@ -60,4 +80,9 @@
     </link>
     <link name="${prefix}finger1">
+      <inertial>
+        <origin xyz="0 0 0" rpy="0 0 0"/>
+        <mass value="0.01"/>
+        <inertia ixx="0.0001" ixy="0.0" ixz="0.0" iyy="0.0001" iyz="0.0" izz="0.0001"/>
+      </inertial>
       <visual>
         <origin rpy="0 0 0" xyz="0 0 0"/>
@@ -77,4 +102,9 @@
     </link>
     <link name="${prefix}finger2">
+      <inertial>
+        <origin xyz="0 0 0" rpy="0 0 0"/>
+        <mass value="0.01"/>
+        <inertia ixx="0.0001" ixy="0.0" ixz="0.0" iyy="0.0001" iyz="0.0" izz="0.0001"/>
+      </inertial>
       <visual>
         <origin rpy="0 0 0" xyz="0 0 0"/>
@@ -93,72 +123,4 @@
       </collision>
     </link>
-    <!-- <link name="${prefix}finger1">
-      <visual>
-        <origin rpy="0 0 0" xyz="0 0 0"/>
-        <geometry>
-          <mesh filename="package://robot_arms/meshes/visual/finger-thin.stl" scale="0.001 0.001 0.001"/>
-        </geometry>
-        <material name="Black">
-          <color rgba="0.1 0.1 0.1 1" />
-        </material>
-      </visual>
-      <collision>
-        <origin rpy="0 0 0" xyz="0 0 0"/>
-        <geometry>
-          <mesh filename="package://robot_arms/meshes/collision/finger-thin.stl" scale="0.001 0.001 0.001"/>
-        </geometry>
-      </collision>
-    </link>
-    <link name="${prefix}finger2">
-      <visual>
-        <origin rpy="0 0 0" xyz="0 0 0"/>
-        <geometry>
-          <mesh filename="package://robot_arms/meshes/visual/finger-thin-prox.stl" scale="0.001 0.001 0.001"/>
-        </geometry>
-        <material name="Black">
-          <color rgba="0.1 0.1 0.1 1" />
-        </material>
-      </visual>
-      <collision>
-        <origin rpy="0 0 0" xyz="0 0 0"/>
-        <geometry>
-          <mesh filename="package://robot_arms/meshes/collision/finger-thin-prox.stl" scale="0.001 0.001 0.001"/>
-        </geometry>
-      </collision>
-    </link> -->
-    <!-- <link name="${prefix}finger1">
-      <visual>
-        <origin rpy="0 0 0" xyz="0 0 0"/>
-        <geometry>
-          <mesh filename="package://robot_arms/meshes/visual/modular_finger.stl" scale="0.001 0.001 0.001"/>
-        </geometry>
-        <material name="Black">
-          <color rgba="0.1 0.1 0.1 1" />
-        </material>
-      </visual>
-      <collision>
-        <origin rpy="0 0 0" xyz="0 0 0"/>
-        <geometry>
-          <mesh filename="package://robot_arms/meshes/collision/modular_finger.stl" scale="0.001 0.001 0.001"/>
-        </geometry>
-      </collision>
-    </link>
-    <link name="${prefix}finger2">
-      <visual>
-        <origin rpy="0 0 0" xyz="0 0 0"/>
-        <geometry>
-          <mesh filename="package://robot_arms/meshes/visual/modular_finger.stl" scale="0.001 0.001 0.001"/>
-        </geometry>
-        <material name="Black">
-          <color rgba="0.1 0.1 0.1 1" />
-        </material>
-      </visual>
-      <collision>
-        <origin rpy="0 0 0" xyz="0 0 0"/>
-        <geometry>
-          <mesh filename="package://robot_arms/meshes/collision/modular_finger.stl" scale="0.001 0.001 0.001"/>
-        </geometry>
-      </collision>
-    </link> -->
     <joint name="${prefix}joint" type="prismatic">
       <origin rpy="0 0 0" xyz="0 0 0.0952"/>
@@ -166,5 +128,5 @@
       <child link="${prefix}jaw1_link"/>
       <axis xyz="1 0 0"/>
-      <limit effort="130" lower="0.0" upper="0.025" velocity="0.15"/>
+      <limit effort="${max_effort}" lower="0.0" upper="${upper_limit}" velocity="0.15"/>
     </joint>
     <joint name="${prefix}base_to_${prefix}jaw2_link" type="prismatic">
@@ -173,5 +135,5 @@
       <child link="${prefix}jaw2_link"/>
       <axis xyz="1 0 0"/>
-      <limit effort="130" lower="0.0" upper="0.025" velocity="0.15"/>
+      <limit effort="${max_effort}" lower="0.0" upper="${upper_limit}" velocity="0.15"/>
       <mimic joint="${prefix}joint" multiplier="1" offset="0"/>
     </joint>
@@ -186,13 +148,4 @@
       <child link="${prefix}finger2"/>
     </joint>
-   <transmission name="${prefix}joint_trans">
-      <type>transmission_interface/SimpleTransmission</type>
-      <joint name="${prefix}joint">
-        <hardwareInterface>hardware_interface/PositionJointInterface</hardwareInterface>
-      </joint>
-      <actuator name="${prefix}joint_motor">
-        <mechanicalReduction>1</mechanicalReduction>
-      </actuator>
-    </transmission>
   </xacro:macro>
 </robot>

File: install/robot_arms/share/robot_arms/urdf/uclv_right_ur5e.urdf.xacro (robot description, xacro)
@@ -1,11 +1,8 @@
 <?xml version="1.0"?>
 <robot xmlns:xacro="http://wiki.ros.org/xacro" name="ur5e">
-   <!-- robot name parameter -->
    <xacro:arg name="name" default="ur5e"/>
-   <!-- import main macro -->
    <xacro:include filename="$(find ur_description)/urdf/ur_macro.xacro"/>
-   <!-- possible 'ur_type' values: ur3, ur3e, ur5, ur5e, ur10, ur10e, ur16e, ur20, ur30 -->
    <xacro:arg name="ur_type" default="ur5e"/>
-   <!-- parameters -->
+   <xacro:include filename="$(find robot_arms)/urdf/robotiq_hande.urdf.xacro" />
    <xacro:arg name="tf_prefix" default="" />
    <xacro:arg name="joint_limit_params" default="$(find ur_description)/config/$(arg ur_type)/joint_limits.yaml"/>
@@ -16,5 +13,4 @@
    <xacro:arg name="safety_pos_margin" default="0.15"/>
    <xacro:arg name="safety_k_position" default="20"/>
-   <!-- create link fixed to the "world" -->
    <link name="world"/>
    <joint name="world_to_table" type="fixed">
@@ -23,8 +19,7 @@
      <origin xyz="0 0 0" rpy="0 0 0"/>
    </joint>
-   <!-- table as base for the UR5e robot -->
    <link name="table">
     <visual>
-      <origin xyz="0 0 0" rpy="0 0 0" />
+      <origin xyz="0 0 0" rpy="0 0 0"/>
       <geometry>
         <mesh filename="package://robot_arms/meshes/visual/myvention_visual.stl" scale="0.001 0.001 0.001"/>
@@ -35,5 +30,5 @@
     </visual>
     <collision>
-      <origin xyz="0 0 0" rpy="0 0 0" />
+      <origin xyz="0 0 0" rpy="0 0 0"/>
       <geometry>
         <mesh filename="package://robot_arms/meshes/collision/myvention_collision.stl" scale="0.001 0.001 0.001"/>
@@ -41,5 +36,4 @@
     </collision>
    </link>
-   <!-- arm -->
    <xacro:ur_robot
      name="ur5e"
@@ -56,7 +50,48 @@
      <origin xyz="-0.188189 0.13575 0.556631" rpy="${3*pi/4} 0 ${-pi/2}" />
    </xacro:ur_robot>
-   <!-- Gazebo Sim ros2_control plugin for ROS 2 Jazzy -->
+   <xacro:robotiq_hande prefix="hande_" origin="$(arg tf_prefix)tool0"/>
+   <ros2_control name="GazeboSimSystem" type="system">
+     <hardware>
+       <plugin>gz_ros2_control/GazeboSimSystem</plugin>
+     </hardware>
+     <joint name="shoulder_pan_joint">
+       <command_interface name="position"/>
+       <state_interface name="position"/>
+       <state_interface name="velocity"/>
+     </joint>
+     <joint name="shoulder_lift_joint">
+       <command_interface name="position"/>
+       <state_interface name="position"/>
+       <state_interface name="velocity"/>
+     </joint>
+     <joint name="elbow_joint">
+       <command_interface name="position"/>
+       <state_interface name="position"/>
+       <state_interface name="velocity"/>
+     </joint>
+     <joint name="wrist_1_joint">
+       <command_interface name="position"/>
+       <state_interface name="position"/>
+       <state_interface name="velocity"/>
+     </joint>
+     <joint name="wrist_2_joint">
+       <command_interface name="position"/>
+       <state_interface name="position"/>
+       <state_interface name="velocity"/>
+     </joint>
+     <joint name="wrist_3_joint">
+       <command_interface name="position"/>
+       <state_interface name="position"/>
+       <state_interface name="velocity"/>
+     </joint>
+     <joint name="hande_joint">
+       <command_interface name="position"/>
+       <state_interface name="position"/>
+       <state_interface name="velocity"/>
+     </joint>
+   </ros2_control>
    <gazebo>
      <plugin filename="libgz_ros2_control-system.so" name="gz_ros2_control::GazeboSimROS2ControlPlugin">
+       <parameters>$(find robot_arms)/config/ros2_controllers.yaml</parameters>
      </plugin>
    </gazebo>

Commit message: giunti iniziali fixati

File: install/robot_arms/share/robot_arms/urdf/robotiq_hande.urdf.xacro (robot description, xacro)
@@ -8,6 +8,72 @@
     <xacro:property name="upper_limit" value="${gripper_props['robotiq_hande']['limits']['upper_stroke']}" />
     <xacro:property name="max_effort" value="${gripper_props['robotiq_hande']['limits']['max_effort']}" />
+    <joint name="${prefix}flange_to_camera_mount" type="fixed">
+      <parent link="${origin}"/>
+      <child link="${prefix}camera_mount_link"/>
+      <origin xyz="0 0 0" rpy="0 0 0"/>
+    </joint>
+    <link name="${prefix}camera_mount_link">
+      <inertial>
+        <mass value="0.08"/>
+        <origin xyz="0 0.028 0.005" rpy="0 0 0"/>
+        <inertia ixx="0.0001" ixy="0.0" ixz="0.0" iyy="0.0001" iyz="0.0" izz="0.0001"/>
+      </inertial>
+      <visual>
+        <origin xyz="0 0 0" rpy="-1.5708 0 0"/>
+        <geometry>
+          <mesh filename="package://robot_arms/meshes/mount/realsenseURflangeSupport.stl" scale="0.001 0.001 0.001"/>
+        </geometry>
+        <material name="MountGray">
+          <color rgba="0.4 0.4 0.4 1.0"/>
+        </material>
+      </visual>
+      <collision>
+        <origin xyz="0 0 0" rpy="-1.5708 0 0"/>
+        <geometry>
+          <mesh filename="package://robot_arms/meshes/mount/realsenseURflangeSupport.stl" scale="0.001 0.001 0.001"/>
+        </geometry>
+      </collision>
+    </link>
+    <gazebo reference="${prefix}camera_mount_link">
+      <visual>
+        <material>
+          <ambient>0.3 0.3 0.3 1.0</ambient>
+          <diffuse>0.4 0.4 0.4 1.0</diffuse>
+          <specular>0.2 0.2 0.2 1.0</specular>
+        </material>
+      </visual>
+    </gazebo>
+    <joint name="${prefix}camera_mount_to_camera" type="fixed">
+      <parent link="${prefix}camera_mount_link"/>
+      <child link="${prefix}camera_link"/>
+      <origin xyz="0 0.0575 0.01145" rpy="0 0 0"/>
+    </joint>
+    <link name="${prefix}camera_link">
+      <inertial>
+        <mass value="0.072"/>
+        <origin xyz="0 0 0" rpy="0 0 0"/>
+        <inertia ixx="0.00005" ixy="0.0" ixz="0.0" iyy="0.00001" iyz="0.0" izz="0.00005"/>
+      </inertial>
+      <visual>
+        <origin xyz="0.005 0 0" rpy="0 0 0"/>
+        <geometry>
+          <mesh filename="package://robot_arms/meshes/camera/d435.dae"/>
+        </geometry>
+      </visual>
+      <collision>
+        <origin xyz="0.005 0 0" rpy="0 0 0"/>
+        <geometry>
+          <box size="0.026 0.090 0.025"/>
+        </geometry>
+      </collision>
+    </link>
+    <joint name="${prefix}camera_to_optical" type="fixed">
+      <parent link="${prefix}camera_link"/>
+      <child link="${prefix}camera_color_optical_frame"/>
+      <origin xyz="0 0 0" rpy="-1.5708 0 -1.5708"/>
+    </joint>
+    <link name="${prefix}camera_color_optical_frame"/>
     <joint name="${prefix}base_to_gripper" type="fixed">
-      <origin rpy="0 0 0" xyz="0 0 0"/>
+      <origin rpy="0 0 0" xyz="0 0 0.005"/>
       <parent link="${origin}"/>
       <child link="${prefix}base_link"/>

File: src/robot_arms/urdf/robotiq_hande.urdf.xacro (robot description, xacro)
@@ -8,6 +8,72 @@
     <xacro:property name="upper_limit" value="${gripper_props['robotiq_hande']['limits']['upper_stroke']}" />
     <xacro:property name="max_effort" value="${gripper_props['robotiq_hande']['limits']['max_effort']}" />
+    <joint name="${prefix}flange_to_camera_mount" type="fixed">
+      <parent link="${origin}"/>
+      <child link="${prefix}camera_mount_link"/>
+      <origin xyz="0 0 0" rpy="0 0 0"/>
+    </joint>
+    <link name="${prefix}camera_mount_link">
+      <inertial>
+        <mass value="0.08"/>
+        <origin xyz="0 0.028 0.005" rpy="0 0 0"/>
+        <inertia ixx="0.0001" ixy="0.0" ixz="0.0" iyy="0.0001" iyz="0.0" izz="0.0001"/>
+      </inertial>
+      <visual>
+        <origin xyz="0 0 0" rpy="-1.5708 0 0"/>
+        <geometry>
+          <mesh filename="package://robot_arms/meshes/mount/realsenseURflangeSupport.stl" scale="0.001 0.001 0.001"/>
+        </geometry>
+        <material name="MountGray">
+          <color rgba="0.4 0.4 0.4 1.0"/>
+        </material>
+      </visual>
+      <collision>
+        <origin xyz="0 0 0" rpy="-1.5708 0 0"/>
+        <geometry>
+          <mesh filename="package://robot_arms/meshes/mount/realsenseURflangeSupport.stl" scale="0.001 0.001 0.001"/>
+        </geometry>
+      </collision>
+    </link>
+    <gazebo reference="${prefix}camera_mount_link">
+      <visual>
+        <material>
+          <ambient>0.3 0.3 0.3 1.0</ambient>
+          <diffuse>0.4 0.4 0.4 1.0</diffuse>
+          <specular>0.2 0.2 0.2 1.0</specular>
+        </material>
+      </visual>
+    </gazebo>
+    <joint name="${prefix}camera_mount_to_camera" type="fixed">
+      <parent link="${prefix}camera_mount_link"/>
+      <child link="${prefix}camera_link"/>
+      <origin xyz="0 0.0575 0.01145" rpy="0 0 0"/>
+    </joint>
+    <link name="${prefix}camera_link">
+      <inertial>
+        <mass value="0.072"/>
+        <origin xyz="0 0 0" rpy="0 0 0"/>
+        <inertia ixx="0.00005" ixy="0.0" ixz="0.0" iyy="0.00001" iyz="0.0" izz="0.00005"/>
+      </inertial>
+      <visual>
+        <origin xyz="0 0 0" rpy="0 0 0"/>
+        <geometry>
+          <mesh filename="package://robot_arms/meshes/camera/d435.dae"/>
+        </geometry>
+      </visual>
+      <collision>
+        <origin xyz="0 0 0" rpy="0 0 0"/>
+        <geometry>
+          <box size="0.026 0.090 0.025"/>
+        </geometry>
+      </collision>
+    </link>
+    <joint name="${prefix}camera_to_optical" type="fixed">
+      <parent link="${prefix}camera_link"/>
+      <child link="${prefix}camera_color_optical_frame"/>
+      <origin xyz="0 0 0" rpy="-1.5708 0 -1.5708"/>
+    </joint>
+    <link name="${prefix}camera_color_optical_frame"/>
     <joint name="${prefix}base_to_gripper" type="fixed">
-      <origin rpy="0 0 0" xyz="0 0 0"/>
+      <origin rpy="0 0 0" xyz="0 0 0.005"/>
       <parent link="${origin}"/>
       <child link="${prefix}base_link"/>

File: src/robot_arms/urdf/uclv_right_ur5e.urdf.xacro (robot description, xacro)
@@ -57,30 +57,30 @@
      <joint name="shoulder_pan_joint">
        <command_interface name="position"/>
-       <state_interface name="position"><param name="initial_value">0.0</param></state_interface>
+       <state_interface name="position"><param name="initial_value">0.7</param></state_interface>
        <state_interface name="velocity"/>
      </joint>
      <joint name="shoulder_lift_joint">
        <command_interface name="position"/>
-       <state_interface name="position"><param name="initial_value">0.0</param></state_interface>
+       <state_interface name="position"><param name="initial_value">0.83</param></state_interface>
        <state_interface name="velocity"/>
      </joint>
      <joint name="elbow_joint">
        <command_interface name="position"/>
-       <state_interface name="position"><param name="initial_value">0.0</param></state_interface>
+       <state_interface name="position"><param name="initial_value">-2.18</param></state_interface>
        <state_interface name="velocity"/>
      </joint>
      <joint name="wrist_1_joint">
        <command_interface name="position"/>
-       <state_interface name="position"><param name="initial_value">0.0</param></state_interface>
+       <state_interface name="position"><param name="initial_value">-1.1</param></state_interface>
        <state_interface name="velocity"/>
      </joint>
      <joint name="wrist_2_joint">
        <command_interface name="position"/>
-       <state_interface name="position"><param name="initial_value">0.0</param></state_interface>
+       <state_interface name="position"><param name="initial_value">2.2</param></state_interface>
        <state_interface name="velocity"/>
      </joint>
      <joint name="wrist_3_joint">
        <command_interface name="position"/>
-       <state_interface name="position"><param name="initial_value">0.0</param></state_interface>
+       <state_interface name="position"><param name="initial_value">0.43</param></state_interface>
        <state_interface name="velocity"/>
      </joint>

Commit message: camera fissata alla giusta distanza dal mount

File: install/robot_arms/share/robot_arms/urdf/robotiq_hande.urdf.xacro (robot description, xacro)
@@ -47,5 +47,5 @@
       <parent link="${prefix}camera_mount_link"/>
       <child link="${prefix}camera_link"/>
-      <origin xyz="0 0.0575 0.01145" rpy="0 0 0"/>
+      <origin xyz="0 0.0575 0.03" rpy="0 0 0"/>
     </joint>
     <link name="${prefix}camera_link">
@@ -56,5 +56,5 @@
       </inertial>
       <visual>
-        <origin xyz="0.005 0 0" rpy="0 0 0"/>
+        <origin xyz="0 0 0" rpy="0 0 0"/>
         <geometry>
           <mesh filename="package://robot_arms/meshes/camera/d435.dae"/>
@@ -62,5 +62,5 @@
       </visual>
       <collision>
-        <origin xyz="0.005 0 0" rpy="0 0 0"/>
+        <origin xyz="0 0 0" rpy="0 0 0"/>
         <geometry>
           <box size="0.026 0.090 0.025"/>

File: src/robot_arms/urdf/robotiq_hande.urdf.xacro (robot description, xacro)
@@ -47,5 +47,5 @@
       <parent link="${prefix}camera_mount_link"/>
       <child link="${prefix}camera_link"/>
-      <origin xyz="0 0.0575 0.01145" rpy="0 0 0"/>
+      <origin xyz="0 0.0575 0.03" rpy="0 0 0"/>
     </joint>
     <link name="${prefix}camera_link">
