Commit message: primo test gazebo

File: install/robot_arms/share/robot_arms/urdf/uclv_right_ur5e.urdf.xacro (robot description, xacro)
@@ -7,6 +7,4 @@
    <!-- possible 'ur_type' values: ur3, ur3e, ur5, ur5e, ur10, ur10e, ur16e, ur20, ur30 -->
    <xacro:arg name="ur_type" default="ur5e"/>
-   <!-- import hande -->
-   <xacro:include filename="$(find robot_arms)/urdf/robotiq_hande.urdf.xacro" />
    <!-- parameters -->
    <xacro:arg name="tf_prefix" default="" />
@@ -18,6 +16,13 @@
    <xacro:arg name="safety_pos_margin" default="0.15"/>
    <xacro:arg name="safety_k_position" default="20"/>
-   <xacro:robotiq_hande prefix="hande_" origin="$(arg tf_prefix)tool0"/>
-   <link name="world">
+   <!-- create link fixed to the "world" -->
+   <link name="world"/>
+   <joint name="world_to_table" type="fixed">
+     <parent link="world"/>
+     <child link="table"/>
+     <origin xyz="0 0 0" rpy="0 0 0"/>
+   </joint>
+   <!-- table as base for the UR5e robot -->
+   <link name="table">
     <visual>
       <origin xyz="0 0 0" rpy="0 0 0" />
@@ -40,5 +45,5 @@
      name="ur5e"
      tf_prefix="$(arg tf_prefix)"
-     parent="world"
+     parent="table"
      joint_limits_parameters_file="$(arg joint_limit_params)"
      kinematics_parameters_file="$(arg kinematics_params)"
@@ -49,5 +54,10 @@
      safety_k_position="$(arg safety_k_position)"
      >
-     <origin xyz="-0.188189 0.13575 0.556631" rpy="${3*pi/4} 0 ${-pi/2}" />          <!-- position robot in the world -->
+     <origin xyz="-0.188189 0.13575 0.556631" rpy="${3*pi/4} 0 ${-pi/2}" />
    </xacro:ur_robot>
+   <!-- Gazebo Sim ros2_control plugin for ROS 2 Jazzy -->
+   <gazebo>
+     <plugin filename="libgz_ros2_control-system.so" name="gz_ros2_control::GazeboSimROS2ControlPlugin">
+     </plugin>
+   </gazebo>
 </robot>

Commit message: gripper completo

File: install/robot_arms/share/robot_arms/urdf/uclv_right_ur5e.urdf.xacro (robot description, xacro)
@@ -90,4 +90,10 @@
        <state_interface name="velocity"/>
      </joint>
+     <joint name="hande_base_to_hande_jaw2_link">
+       <param name="mimic">hande_joint</param>
+       <param name="multiplier">1.0</param>
+       <state_interface name="position"/>
+       <state_interface name="velocity"/>
+     </joint>
    </ros2_control>
    <gazebo>

Commit message: aggiunta scacchiera nella scena

File: install/robot_arms/share/robot_arms/urdf/uclv_right_ur5e.urdf.xacro (robot description, xacro)
@@ -36,4 +36,30 @@
     </collision>
    </link>
+   <joint name="table_to_chessboard" type="fixed">
+     <parent link="table"/>
+     <child link="chessboard"/>
+     <origin xyz="-0.5 -0.15 0" rpy="0 0 -1.5708"/>
+   </joint>
+   <link name="chessboard">
+     <inertial>
+       <mass value="1.5"/>
+       <inertia ixx="0.03" ixy="0.0" ixz="0.0" iyy="0.03" iyz="0.0" izz="0.06"/>
+     </inertial>
+     <visual>
+       <origin xyz="0 0 0" rpy="0 0 0"/>
+       <geometry>
+         <mesh filename="package://robot_arms/meshes/scacchi/chessboard.stl" scale="0.005 0.005 0.005"/>
+       </geometry>
+       <material name="Wood">
+         <color rgba="0.76 0.60 0.42 1.0"/>
+       </material>
+     </visual>
+     <collision>
+       <origin xyz="0 0 0" rpy="0 0 0"/>
+       <geometry>
+         <mesh filename="package://robot_arms/meshes/scacchi/chessboard.stl" scale="0.005 0.005 0.005"/>
+       </geometry>
+     </collision>
+   </link>
    <xacro:ur_robot
      name="ur5e"
@@ -57,30 +83,42 @@
      <joint name="shoulder_pan_joint">
        <command_interface name="position"/>
-       <state_interface name="position"/>
+       <state_interface name="position">
+         <param name="initial_value">0.0</param>
+       </state_interface>
        <state_interface name="velocity"/>
      </joint>
      <joint name="shoulder_lift_joint">
        <command_interface name="position"/>
-       <state_interface name="position"/>
+       <state_interface name="position">
+         <param name="initial_value">0.0</param>
+       </state_interface>
        <state_interface name="velocity"/>
      </joint>
      <joint name="elbow_joint">
        <command_interface name="position"/>
-       <state_interface name="position"/>
+       <state_interface name="position">
+         <param name="initial_value">0.0</param>
+       </state_interface>
        <state_interface name="velocity"/>
      </joint>
      <joint name="wrist_1_joint">
        <command_interface name="position"/>
-       <state_interface name="position"/>
+       <state_interface name="position">
+         <param name="initial_value">0.0</param>
+       </state_interface>
        <state_interface name="velocity"/>
      </joint>
      <joint name="wrist_2_joint">
        <command_interface name="position"/>
-       <state_interface name="position"/>
+       <state_interface name="position">
+         <param name="initial_value">0.0</param>
+       </state_interface>
        <state_interface name="velocity"/>
      </joint>
      <joint name="wrist_3_joint">
        <command_interface name="position"/>
-       <state_interface name="position"/>
+       <state_interface name="position">
+         <param name="initial_value">0.0</param>
+       </state_interface>
        <state_interface name="velocity"/>
      </joint>

Commit message: scacchiera completa di pezzi

File: install/robot_arms/share/robot_arms/urdf/uclv_right_ur5e.urdf.xacro (robot description, xacro)
@@ -36,30 +36,4 @@
     </collision>
    </link>
-   <joint name="table_to_chessboard" type="fixed">
-     <parent link="table"/>
-     <child link="chessboard"/>
-     <origin xyz="-0.5 -0.15 0" rpy="0 0 -1.5708"/>
-   </joint>
-   <link name="chessboard">
-     <inertial>
-       <mass value="1.5"/>
-       <inertia ixx="0.03" ixy="0.0" ixz="0.0" iyy="0.03" iyz="0.0" izz="0.06"/>
-     </inertial>
-     <visual>
-       <origin xyz="0 0 0" rpy="0 0 0"/>
-       <geometry>
-         <mesh filename="package://robot_arms/meshes/scacchi/chessboard.stl" scale="0.005 0.005 0.005"/>
-       </geometry>
-       <material name="Wood">
-         <color rgba="0.76 0.60 0.42 1.0"/>
-       </material>
-     </visual>
-     <collision>
-       <origin xyz="0 0 0" rpy="0 0 0"/>
-       <geometry>
-         <mesh filename="package://robot_arms/meshes/scacchi/chessboard.stl" scale="0.005 0.005 0.005"/>
-       </geometry>
-     </collision>
-   </link>
    <xacro:ur_robot
      name="ur5e"
@@ -83,42 +57,30 @@
      <joint name="shoulder_pan_joint">
        <command_interface name="position"/>
-       <state_interface name="position">
-         <param name="initial_value">0.0</param>
-       </state_interface>
+       <state_interface name="position"><param name="initial_value">0.0</param></state_interface>
        <state_interface name="velocity"/>
      </joint>
      <joint name="shoulder_lift_joint">
        <command_interface name="position"/>
-       <state_interface name="position">
-         <param name="initial_value">0.0</param>
-       </state_interface>
+       <state_interface name="position"><param name="initial_value">0.0</param></state_interface>
        <state_interface name="velocity"/>
      </joint>
      <joint name="elbow_joint">
        <command_interface name="position"/>
-       <state_interface name="position">
-         <param name="initial_value">0.0</param>
-       </state_interface>
+       <state_interface name="position"><param name="initial_value">0.0</param></state_interface>
        <state_interface name="velocity"/>
      </joint>
      <joint name="wrist_1_joint">
        <command_interface name="position"/>
-       <state_interface name="position">
-         <param name="initial_value">0.0</param>
-       </state_interface>
+       <state_interface name="position"><param name="initial_value">0.0</param></state_interface>
        <state_interface name="velocity"/>
      </joint>
      <joint name="wrist_2_joint">
        <command_interface name="position"/>
-       <state_interface name="position">
-         <param name="initial_value">0.0</param>
-       </state_interface>
+       <state_interface name="position"><param name="initial_value">0.0</param></state_interface>
        <state_interface name="velocity"/>
      </joint>
      <joint name="wrist_3_joint">
        <command_interface name="position"/>
-       <state_interface name="position">
-         <param name="initial_value">0.0</param>
-       </state_interface>
+       <state_interface name="position"><param name="initial_value">0.0</param></state_interface>
        <state_interface name="velocity"/>
      </joint>

Commit message: DA CONTROLLARE: aggiunti colori ma la scacchiera mo affonda

File: install/robot_arms/share/robot_arms/urdf/uclv_right_ur5e.urdf.xacro (robot description, xacro)
@@ -36,4 +36,32 @@
     </collision>
    </link>
+   <link name="wall_link">
+     <visual>
+       <origin xyz="0 0 1.0" rpy="0 0 0"/>
+       <geometry>
+         <box size="3.0 0.1 2.0"/> </geometry>
+       <material name="WallWhite">
+         <color rgba="0.9 0.9 0.9 1.0"/>
+       </material>
+     </visual>
+     <collision>
+       <origin xyz="0 0 1.0" rpy="0 0 0"/>
+       <geometry>
+         <box size="3.0 0.1 2.0"/>
+       </geometry>
+     </collision>
+   </link>
+   <joint name="table_to_wall" type="fixed">
+     <parent link="table"/>
+     <child link="wall_link"/>
+     <origin xyz="0 0.55 0" rpy="0 0 0"/>
+   </joint>
+   <gazebo reference="wall_link">
+     <visual>
+       <material>
+         <ambient>0.9 0.9 0.95 1.0</ambient> <diffuse>0.9 0.9 0.95 1.0</diffuse>
+       </material>
+     </visual>
+   </gazebo>
    <xacro:ur_robot
      name="ur5e"

File: src/robot_arms/urdf/chessboard.urdf.xacro (robot description, xacro)
@@ -1,5 +1,5 @@
 <?xml version="1.0"?>
 <robot xmlns:xacro="http://wiki.ros.org/xacro" name="chessboard">
-  <link name="chessboard_link">
+<link name="chessboard_link">
     <inertial>
       <origin xyz="0 0 0.005" rpy="0 0 0"/>
@@ -8,14 +8,11 @@
     </inertial>
     <visual>
-      <origin xyz="0 0 0" rpy="0 0 0"/>
+      <origin xyz="0 0 0.005" rpy="1.5708 0 0"/>
       <geometry>
-        <mesh filename="package://robot_arms/meshes/scacchi/chessboard.stl" scale="0.005 0.005 0.005"/>
+        <mesh filename="package://robot_arms/meshes/scacchi/chessboard.obj" scale="1 1 1"/>
       </geometry>
-      <material name="Wood">
-        <color rgba="0.76 0.60 0.42 1.0"/>
-      </material>
-    </visual>
+      </visual>
     <collision>
-      <origin xyz="0 0 0.005" rpy="0 0 0"/>
+      <origin xyz="0 0 0.005" rpy="1.5708 0 0"/>
       <geometry>
         <box size="0.51 0.51 0.01"/>
@@ -52,4 +49,10 @@
     <origin xyz="0.28 0.23 0.013" rpy="0 0 0"/>
   </joint>
+  <link name="a1_square_link"/>
+  <joint name="aruco_to_a1" type="fixed">
+    <parent link="aruco_marker_link"/>
+    <child link="a1_square_link"/>
+    <origin xyz="0.0685 0.066 0" rpy="0 0 0"/>
+  </joint>
   <gazebo reference="aruco_marker_link">
     <visual>

Commit message: scacchiera aggiustata, da sistemare lo spawn dei pezzi

File: install/robot_arms/share/robot_arms/urdf/uclv_right_ur5e.urdf.xacro (robot description, xacro)
@@ -38,5 +38,5 @@
    <link name="wall_link">
      <visual>
-       <origin xyz="0 0 1.0" rpy="0 0 0"/>
+       <origin xyz="0 0 0.0" rpy="0 0 0"/>
        <geometry>
          <box size="3.0 0.1 2.0"/> </geometry>
@@ -46,5 +46,5 @@
      </visual>
      <collision>
-       <origin xyz="0 0 1.0" rpy="0 0 0"/>
+       <origin xyz="0 0 0.0" rpy="0 0 0"/>
        <geometry>
          <box size="3.0 0.1 2.0"/>

File: src/robot_arms/urdf/chessboard.urdf.xacro (robot description, xacro)
@@ -1,20 +1,20 @@
 <?xml version="1.0"?>
 <robot xmlns:xacro="http://wiki.ros.org/xacro" name="chessboard">
-<link name="chessboard_link">
+  <link name="chessboard_link">
     <inertial>
-      <origin xyz="0 0 0.005" rpy="0 0 0"/>
+      <origin xyz="0 0 0.0075" rpy="0 0 0"/>
       <mass value="1.5"/>
       <inertia ixx="0.03" ixy="0.0" ixz="0.0" iyy="0.03" iyz="0.0" izz="0.06"/>
     </inertial>
     <visual>
-      <origin xyz="0 0 0.005" rpy="1.5708 0 0"/>
+      <origin xyz="0 0 0" rpy="1.5708 0 0"/>
       <geometry>
         <mesh filename="package://robot_arms/meshes/scacchi/chessboard.obj" scale="1 1 1"/>
       </geometry>
-      </visual>
+    </visual>
     <collision>
-      <origin xyz="0 0 0.005" rpy="1.5708 0 0"/>
+      <origin xyz="0 0 0" rpy="0 0 0"/>
       <geometry>
-        <box size="0.51 0.51 0.01"/>
+        <box size="0.51 0.51 0.015"/>
       </geometry>
     </collision>
@@ -23,29 +23,17 @@
     <mu1>1.0</mu1>
     <mu2>1.0</mu2>
-    <kp>1000000.0</kp>
-    <kd>1.0</kd>
   </gazebo>
-<link name="aruco_marker_link">
-    <inertial>
-      <mass value="0.01"/>
-      <origin xyz="0 0 0" rpy="0 0 0"/>
-      <inertia ixx="0.00001" ixy="0" ixz="0" iyy="0.00001" iyz="0" izz="0.00001"/>
-    </inertial>
+  <link name="aruco_marker_link">
     <visual>
-      <origin xyz="0 0 0" rpy="0 0 0"/>
-      <geometry>
-        <box size="0.05 0.05 0.001"/> </geometry>
-    </visual>
-    <collision>
       <origin xyz="0 0 0" rpy="0 0 0"/>
       <geometry>
         <box size="0.05 0.05 0.001"/>
       </geometry>
-    </collision>
+    </visual>
   </link>
   <joint name="chessboard_to_aruco" type="fixed">
     <parent link="chessboard_link"/>
     <child link="aruco_marker_link"/>
-    <origin xyz="0.28 0.23 0.013" rpy="0 0 0"/>
+    <origin xyz="0.28 0.23 0.0155" rpy="0 0 0"/>
   </joint>
   <link name="a1_square_link"/>
@@ -53,5 +41,5 @@
     <parent link="aruco_marker_link"/>
     <child link="a1_square_link"/>
-    <origin xyz="0.0685 0.066 0" rpy="0 0 0"/>
+    <origin xyz="-0.0805 -0.0305 0" rpy="0 0 0"/>
   </joint>
   <gazebo reference="aruco_marker_link">
@@ -64,6 +52,4 @@
           <metal>
             <albedo_map>file://$(find robot_arms)/materials/textures/aruco_0.png</albedo_map>
-            <roughness>1.0</roughness>
-            <metalness>0.0</metalness>
           </metal>
         </pbr>
