Commit message: aggiunto aruco alla scena

File: src/robot_arms/urdf/chessboard.urdf.xacro (robot description, xacro)
@@ -29,3 +29,42 @@
     <kd>1.0</kd>
   </gazebo>
+<link name="aruco_marker_link">
+    <inertial>
+      <mass value="0.01"/>
+      <origin xyz="0 0 0" rpy="0 0 0"/>
+      <inertia ixx="0.00001" ixy="0" ixz="0" iyy="0.00001" iyz="0" izz="0.00001"/>
+    </inertial>
+    <visual>
+      <origin xyz="0 0 0" rpy="0 0 0"/>
+      <geometry>
+        <box size="0.05 0.05 0.001"/> </geometry>
+    </visual>
+    <collision>
+      <origin xyz="0 0 0" rpy="0 0 0"/>
+      <geometry>
+        <box size="0.05 0.05 0.001"/>
+      </geometry>
+    </collision>
+  </link>
+  <joint name="chessboard_to_aruco" type="fixed">
+    <parent link="chessboard_link"/>
+    <child link="aruco_marker_link"/>
+    <origin xyz="0.28 0.23 0.013" rpy="0 0 0"/>
+  </joint>
+  <gazebo reference="aruco_marker_link">
+    <visual>
+      <material>
+        <diffuse>1 1 1 1</diffuse>
+        <ambient>1 1 1 1</ambient>
+        <emissive>0.1 0.1 0.1 1</emissive>
+        <pbr>
+          <metal>
+            <albedo_map>file://$(find robot_arms)/materials/textures/aruco_0.png</albedo_map>
+            <roughness>1.0</roughness>
+            <metalness>0.0</metalness>
+          </metal>
+        </pbr>
+      </material>
+    </visual>
+  </gazebo>
 </robot>
