Commit message: movimento e2e4 funzionante

File: src/robot_arms/urdf/chess_piece.urdf.xacro (robot description, xacro)
@@ -5,10 +5,10 @@
   <xacro:arg name="piece_type" default="p"/>
   <xacro:property name="piece_data" value="${dict(
-      p=dict(vx=0.0,    vy=0.0, vz=0.0, c_rad=0.013, c_len=0.05,  c_z=0.025),
-      r=dict(vx=0.0,    vy=0.0, vz=0.0, c_rad=0.015, c_len=0.055, c_z=0.0275),
-      n=dict(vx=0.0,    vy=0.0, vz=0.0, c_rad=0.015, c_len=0.06,  c_z=0.03),
-      b=dict(vx=0.0,    vy=0.0, vz=0.0, c_rad=0.015, c_len=0.07,  c_z=0.035),
-      q=dict(vx=0.0,    vy=0.0, vz=0.0, c_rad=0.018, c_len=0.08,  c_z=0.04),
-      k=dict(vx=0.0,    vy=0.0, vz=0.0, c_rad=0.018, c_len=0.09,  c_z=0.045)
+      p=dict(vx=0.0,    vy=0.0, vz=0.0, c_rad=0.0085, c_len=0.045, c_z=0.0225),
+      r=dict(vx=0.0,    vy=0.0, vz=0.0, c_rad=0.0110, c_len=0.055, c_z=0.0275),
+      n=dict(vx=0.0,    vy=0.0, vz=0.0, c_rad=0.0110, c_len=0.060, c_z=0.0300),
+      b=dict(vx=0.0,    vy=0.0, vz=0.0, c_rad=0.0110, c_len=0.070, c_z=0.0350),
+      q=dict(vx=0.0,    vy=0.0, vz=0.0, c_rad=0.0120, c_len=0.080, c_z=0.0400),
+      k=dict(vx=0.0,    vy=0.0, vz=0.0, c_rad=0.0120, c_len=0.090, c_z=0.0450)
   )}"/>
   <xacro:property name="data" value="${piece_data['$(arg piece_type)']}"/>

File: src/robot_arms/urdf/robotiq_hande.urdf.xacro (robot description, xacro)
@@ -194,5 +194,5 @@
       <child link="${prefix}jaw1_link"/>
       <axis xyz="1 0 0"/>
-      <limit effort="${max_effort}" lower="0.0" upper="${upper_limit}" velocity="0.15"/>
+      <limit effort="${max_effort}" lower="-0.015" upper="${upper_limit}" velocity="0.15"/>
     </joint>
     <joint name="${prefix}base_to_${prefix}jaw2_link" type="prismatic">
@@ -201,6 +201,5 @@
       <child link="${prefix}jaw2_link"/>
       <axis xyz="1 0 0"/>
-      <limit effort="${max_effort}" lower="0.0" upper="${upper_limit}" velocity="0.15"/>
-      <mimic joint="${prefix}joint" multiplier="1" offset="0"/>
+      <limit effort="${max_effort}" lower="-0.015" upper="${upper_limit}" velocity="0.15"/>
     </joint>
     <joint name="${prefix}jaw1_to_finger1" type="fixed">
@@ -214,4 +213,16 @@
       <child link="${prefix}finger2"/>
     </joint>
+    <gazebo reference="${prefix}finger1">
+      <mu1>5.0</mu1>
+      <mu2>5.0</mu2>
+      <kp>1000000.0</kp>
+      <kd>10.0</kd>
+    </gazebo>
+    <gazebo reference="${prefix}finger2">
+      <mu1>5.0</mu1>
+      <mu2>5.0</mu2>
+      <kp>1000000.0</kp>
+      <kd>10.0</kd>
+    </gazebo>
   </xacro:macro>
 </robot>

File: src/robot_arms/urdf/uclv_right_ur5e.urdf.xacro (robot description, xacro)
@@ -85,41 +85,40 @@
      <joint name="shoulder_pan_joint">
        <command_interface name="position"/>
-       <state_interface name="position"><param name="initial_value">0.7</param></state_interface>
+       <state_interface name="position"><param name="initial_value">0.335</param></state_interface>
        <state_interface name="velocity"/>
      </joint>
      <joint name="shoulder_lift_joint">
        <command_interface name="position"/>
-       <state_interface name="position"><param name="initial_value">0.83</param></state_interface>
+       <state_interface name="position"><param name="initial_value">0.771</param></state_interface>
        <state_interface name="velocity"/>
      </joint>
      <joint name="elbow_joint">
        <command_interface name="position"/>
-       <state_interface name="position"><param name="initial_value">-2.18</param></state_interface>
+       <state_interface name="position"><param name="initial_value">-2.282</param></state_interface>
        <state_interface name="velocity"/>
      </joint>
      <joint name="wrist_1_joint">
        <command_interface name="position"/>
-       <state_interface name="position"><param name="initial_value">-1.1</param></state_interface>
+       <state_interface name="position"><param name="initial_value">-0.377</param></state_interface>
        <state_interface name="velocity"/>
      </joint>
      <joint name="wrist_2_joint">
        <command_interface name="position"/>
-       <state_interface name="position"><param name="initial_value">2.2</param></state_interface>
+       <state_interface name="position"><param name="initial_value">2.302</param></state_interface>
        <state_interface name="velocity"/>
      </joint>
      <joint name="wrist_3_joint">
        <command_interface name="position"/>
-       <state_interface name="position"><param name="initial_value">0.43</param></state_interface>
+       <state_interface name="position"><param name="initial_value">1.113</param></state_interface>
        <state_interface name="velocity"/>
      </joint>
      <joint name="hande_joint">
        <command_interface name="position"/>
-       <state_interface name="position"/>
+       <state_interface name="position"><param name="initial_value">0.0</param></state_interface>
        <state_interface name="velocity"/>
      </joint>
      <joint name="hande_base_to_hande_jaw2_link">
-       <param name="mimic">hande_joint</param>
-       <param name="multiplier">1.0</param>
-       <state_interface name="position"/>
+       <command_interface name="position"/>
+       <state_interface name="position"><param name="initial_value">0.0</param></state_interface>
        <state_interface name="velocity"/>
      </joint>

Commit message: velocizzato movimento simulazione e aggiornato gitignore

File: src/robot_arms/urdf/chess_piece.urdf.xacro (robot description, xacro)
@@ -28,16 +28,7 @@
       </material>
     </visual>
-    <collision>
-      <origin xyz="0 0 ${data['c_z']}" rpy="0 0 0"/>
-      <geometry>
-        <cylinder radius="${data['c_rad']}" length="${data['c_len']}"/>
-      </geometry>
-    </collision>
   </link>
-  <gazebo reference="piece_base_link">
-    <mu1>1.5</mu1>
-    <mu2>1.5</mu2>
-    <kp>1000000.0</kp>
-    <kd>1.0</kd>
+  <gazebo>
+    <static>true</static>
   </gazebo>
 </robot>
