Commit message: movimento e2e4 moveit2

File: src/robot_arms/urdf/robotiq_hande.urdf.xacro (robot description, xacro)
@@ -212,4 +212,11 @@
       <parent link="${prefix}jaw2_link"/>
       <child link="${prefix}finger2"/>
+    </joint>
+    <!-- Frame TCP esatto al centro dei polpastrelli della pinza (usato da MoveIt 2 per IK e traiettorie cartesiane) -->
+    <link name="${prefix}tcp_link"/>
+    <joint name="${prefix}tool0_to_tcp" type="fixed">
+      <origin rpy="0 0 0" xyz="0 0 0.225"/>
+      <parent link="${origin}"/>
+      <child link="${prefix}tcp_link"/>
     </joint>
     <gazebo reference="${prefix}finger1">
